File: code/SuperHoop_PCB/SUPERHOOP.sch (EAGLE design)
At the start: 11 parts, among them CON1 Battery_lithium 3.7v (3x), CON2 TOUCH_INPUT, CON3 LED_STRING_OUTPUT, CON4 ADXL335_BBOARD_V2, CON5 ISP-AVR_6P, IC1 MEGA8-P

Commit message: final changes from Sunday
Saved Eagle files, shortened delay between pattern cycles to ~5 seconds
Parts:
- removed QF1: 8M10AHC49T, crystal:8M10AHC49T
- added X1: (no value), crystal:CRYSTALHC49S
Connections:
- net GND: no longer QF1.2
- net MISO: now also IC1.PB4(MISO)
- net MOSI: now also IC1.PB3(MOSI/OC2)
- net SCK: now also IC1.PB5(SCK)
- net XTAL1: now also X1.2; no longer QF1.1
- net XTAL2: now also X1.1; no longer QF1.3
Changed lines of the file:
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@@
 <part name="IC1" library="atmel" deviceset="MEGA8-P" device=""/>
 <part name="CON1" library="daneagle_db" deviceset="HEADER_2X1" device="_2.54" value="Battery_lithium 3.7v (3x)"/>
-<part name="QF1" library="crystal" deviceset="8M10AHC49T" device=""/>
 <part name="CON3" library="daneagle_db" deviceset="HEADER_3X1" device="" value="LED_STRING_OUTPUT"/>
 <part name="C1" library="rcl" deviceset="C-US" device="025-024X044"/>
@@
 <part name="CON2" library="daneagle_db" deviceset="HEADER_2X1" device="_2.54" value="TOUCH_INPUT"/>
 <part name="CON5" library="daneagle_db" deviceset="ISP-AVR" device="_6P"/>
+<part name="X1" library="crystal" deviceset="CRYSTAL" device="HC49S"/>
 </parts>
 <sheets>
@@
 <instance part="IC1" gate="G$1" x="109.22" y="144.78"/>
 <instance part="CON1" gate="G$1" x="223.52" y="180.34"/>
-<instance part="QF1" gate="G$1" x="66.04" y="152.4" rot="R270"/>
 <instance part="CON3" gate="G$1" x="226.06" y="152.4"/>
 <instance part="C1" gate="G$1" x="50.8" y="160.02"/>
@@
 <instance part="CON2" gate="G$1" x="162.56" y="187.96"/>
 <instance part="CON5" gate="G$1" x="154.94" y="76.2"/>
+<instance part="X1" gate="G$1" x="66.04" y="152.4" rot="R90"/>
 </instances>
 <busses>
@@
 </segment>
 <segment>
-<pinref part="QF1" gate="G$1" pin="2"/>
 <wire x1="60.96" y1="152.4" x2="50.8" y2="152.4" width="0.1524" layer="91"/>
 <pinref part="C1" gate="G$1" pin="2"/>
@@
 <net name="XTAL1" class="0">
 <segment>
-<pinref part="QF1" gate="G$1" pin="1"/>
 <pinref part="IC1" gate="G$1" pin="PB6(XTAL1/TOSC1)"/>
 <wire x1="66.04" y1="154.94" x2="86.36" y2="154.94" width="0.1524" layer="91"/>
@@
 <wire x1="50.8" y1="165.1" x2="66.04" y2="165.1" width="0.1524" layer="91"/>
 <wire x1="66.04" y1="165.1" x2="66.04" y2="154.94" width="0.1524" layer="91"/>
+<label x="73.66" y="154.94" size="1.778" layer="95"/>
+<pinref part="X1" gate="G$1" pin="2"/>
 <junction x="66.04" y="154.94"/>
-<label x="73.66" y="154.94" size="1.778" layer="95"/>
 </segment>
 </net>
 <net name="XTAL2" class="0">
 <segment>
-<pinref part="QF1" gate="G$1" pin="3"/>
 <pinref part="IC1" gate="G$1" pin="PB7(XTAL2/TOSC2)"/>
 <wire x1="66.04" y1="149.86" x2="86.36" y2="149.86" width="0.1524" layer="91"/>
 <wire x1="66.04" y1="149.86" x2="66.04" y2="139.7" width="0.1524" layer="91"/>
-<junction x="66.04" y="149.86"/>
 <pinref part="C2" gate="G$1" pin="1"/>
 <wire x1="66.04" y1="139.7" x2="50.8" y2="139.7" width="0.1524" layer="91"/>
 <wire x1="50.8" y1="139.7" x2="50.8" y2="142.24" width="0.1524" layer="91"/>
 <label x="73.66" y="149.86" size="1.778" layer="95"/>
+<pinref part="X1" gate="G$1" pin="1"/>
+<junction x="66.04" y="149.86"/>
 </segment>
 </net>
@@
 <label x="134.62" y="78.74" size="1.778" layer="95"/>
 </segment>
+<segment>
+<pinref part="IC1" gate="G$1" pin="PB4(MISO)"/>
+<wire x1="144.78" y1="116.84" x2="134.62" y2="116.84" width="0.1524" layer="91"/>
+<label x="139.7" y="116.84" size="1.778" layer="95"/>
+</segment>
 </net>
 <net name="SCK" class="0">
@@
 <label x="134.62" y="76.2" size="1.778" layer="95"/>
 </segment>
+<segment>
+<pinref part="IC1" gate="G$1" pin="PB5(SCK)"/>
+<wire x1="144.78" y1="114.3" x2="134.62" y2="114.3" width="0.1524" layer="91"/>
+<label x="139.7" y="114.3" size="1.778" layer="95"/>
+</segment>
 </net>
 <net name="RST" class="0">
@@
 <label x="170.18" y="76.2" size="1.778" layer="95"/>
 </segment>
-</net>
+<segment>
+<pinref part="IC1" gate="G$1" pin="PB3(MOSI/OC2)"/>
+<wire x1="144.78" y1="119.38" x2="134.62" y2="119.38" width="0.1524" layer="91"/>
+<label x="139.7" y="119.38" size="1.778" layer="95"/>
+</segment>
+</net>
